File: E-INK Watch/E-INK Watch.kicad_sch (KiCad schematic)
At the start: 13 parts, among them J1 Conn_01x03_Female, J2 USB_B_Micro, U1 PIC18F27J53_ISS, U2 DPS310, Y1 32.768kHz

Commit message: Cleaned up schemtic and pcb
Parts:
- removed J1: Conn_01x03_Female, e-ink:PinHeader_3x2.54_SMD_90deg, symbol Connector:Conn_01x03_Female
- added J1: Conn_01x04_Female, e-ink:HARWIN_M20-7910442R, symbol Connector:Conn_01x04_Female
Connections:
- net +5V: no longer U1.4 (RA2/AN2)
- net BATT_OFF: now also U1.3 (RA1/AN1); no longer U1.2 (RA0/AN0)
- net BATT_V: now also U1.4 (RA2/AN2); no longer U1.3 (RA1/AN1)
- net GND: now also J1.1 (Pin_1)
- net ISCPCLK: now also J1.2 (Pin_2)
- net ISCPDAT: now also J1.3 (Pin_3)
- net ~{MCLR}: now also J1.4 (Pin_4)
- new net USB_IN: U1.2 (RA0/AN0)
Other:
- sheet Power ports: added USB_IN; removed none
- note removed: "Double check ADC pin and RES# is ok/what it do"
- note removed: "Here put pull up to keep n-channel high"
- note removed: "Hook up external temp sense to e ink screen too"
- note removed: "pull up? pull down? IDK"
- moved on the sheet: J2, R2
