File: E-INK Watch/E-INK Watch.kicad_sch (KiCad schematic)
At the start: 13 parts, among them J1 Conn_01x04_Female, J2 USB_B_Micro, U1 PIC18F27J53_ISS, U2 DPS310, Y1 32.768kHz

Commit message: Completed PCB and gerber files
Parts:
- removed C4: 100nF, Capacitor_SMD:C_0603_1608Metric_Pad1.08x0.95mm_HandSolder, symbol Device:C_Small
- added C6: 100nF, Capacitor_SMD:C_0603_1608Metric_Pad1.08x0.95mm_HandSolder, symbol Device:C_Small
- J2: footprint e-ink:AMPHENOL_10118193-0001LF -> Connector_USB:USB_Micro-B_Molex-105017-0001
- renumbered C22 to C1, C1 to C2, C2 to C3, C3 to C4
Connections:
- net +3.3V: now also C6.1
- net GND: now also C6.2
- net BATT_OFF: no longer names the net of U1.3 (RA1/AN1)
- net D/C# renamed D/C
- net RES# renamed RES
- no-connect marks 8 -> 9
Other:
- sheet Power ports: added none; removed BATT_OFF
- sheet Screen ports: added D/C, RES; removed D/C#, RES#
- moved on the sheet: C3, C4, R1, Y1
