File: E-INK Watch/power.kicad_sch (KiCad schematic)
At the start: 18 parts, among them J3 JST PH, Q1 DMG2305UX-13, T1 BSS806NEH6327XTSA1, U3 MCP73831-2-OT, U4 S-1318B33-M5T1U4

Commit message: Cleaned up schemtic and pcb
Parts:
- removed C10: 0.1uF, Capacitor_SMD:C_0603_1608Metric_Pad1.08x0.95mm_HandSolder, symbol Device:C
- removed R7: 328K 0.1%, Resistor_SMD:R_0603_1608Metric_Pad0.98x0.95mm_HandSolder, symbol Device:R_US
- removed R8: 820k 0.1%, Resistor_SMD:R_0603_1608Metric_Pad0.98x0.95mm_HandSolder, symbol Device:R_US
- added C10: 0.1uF, Capacitor_SMD:C_0603_1608Metric_Pad1.08x0.95mm_HandSolder, symbol Device:C_Small
- added R12: 510k 0.1%, Resistor_SMD:R_0603_1608Metric_Pad0.98x0.95mm_HandSolder, symbol Device:R_Small
- added R4: 328k 0.1%, Resistor_SMD:R_0603_1608Metric_Pad0.98x0.95mm_HandSolder, symbol Device:R_Small
- added R7: 820k 0.1%, Resistor_SMD:R_0603_1608Metric_Pad0.98x0.95mm_HandSolder, symbol Device:R_Small
- added R8: 340k 0.1%, Resistor_SMD:R_0603_1608Metric_Pad0.98x0.95mm_HandSolder, symbol Device:R_Small
Connections:
- net +5V: now also R8.2
- net +BATT: now also R4.2
- net BATT_V: now also C10.1, R4.1, R7.2
- net GND: now also C10.2, R12.1, R7.1
- new net USB_IN: R12.2, R8.1
Other:
- note added: "5V -> 3.0V"
- note added: "Disconnects load from battery if voltage gets too low"
- note added: "Switching/Protection/Regulation"
- note added: "USB Detection"
- note removed: "Listen to Jack's Warning"
- moved on the sheet: C6, C7, C8, C9, D2, D3, D4, J3, Q1, R3, R5, R6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
