File: E-INK Watch/power.kicad_sch (KiCad schematic)
At the start: 20 parts, among them J3 JST PH, Q1 DMG2305UX-13, T1 BSS806NEH6327XTSA1, U3 MCP73831-2-OT, U4 S-1318B33-M5T1U4

Commit message: Completed PCB and gerber files
Parts:
- removed T1: BSS806NEH6327XTSA1, e-ink:DIO_BB914E6327HTSA1, symbol MMBF170:MMBF170
- D2: renamed from D3; value SD103AWS-TP -> SD103AW-13-F; footprint e-ink:SOD2512X115N -> Diode_SMD:D_SOD-123
- R3: renamed from R5; value 150 -> 150R
- renumbered C9 to C10, C10 to C11, C6 to C7, C7 to C8, C8 to C9, D2 to D1, D4 to D3, R3 to R4, R6 to R5, R4 to R6, R12 to R9
Connections:
- net at C9.1, D2.1 (K), U4.1 (IN)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: now also Q1.2
Other:
- note removed: "Disconnects load from battery if voltage gets too low"
