File: E-INK Watch/screen.kicad_sch (KiCad schematic)
At the start: 20 parts, among them J4 EINK, Q2 AO3418

Commit message: Cleaned up schemtic and pcb
Parts:
- C11: value 1uF -> 4.7uF
Other:
- moved on the sheet: C15, C16, C17, C18, C19, C20, C21, J4
