File: E-INK Watch/screen.kicad_sch (KiCad schematic)
At the start: 20 parts, among them J4 EINK, Q2 AO3418

Commit message: Completed PCB and gerber files
Parts:
- removed C13: 1uF, Capacitor_SMD:C_0603_1608Metric_Pad1.08x0.95mm_HandSolder, symbol Device:C_Small
- removed R9: 0R, Resistor_SMD:R_0603_1608Metric_Pad0.98x0.95mm_HandSolder, symbol Device:R_Small
- added C22, C23: 4.7uF, Capacitor_SMD:C_0603_1608Metric_Pad1.08x0.95mm_HandSolder, symbol Device:C_Small
- added C24: 1uF, Capacitor_SMD:C_0603_1608Metric_Pad1.08x0.95mm_HandSolder, symbol Device:C_Small
- C13: renamed from C12; value 1uF -> 4.7uF
- C17, C19, C21: value 1uF -> 4.7uF
- L1: value 47uH -> 10uH
- R11: value 2R2 -> 0.47R
- renumbered C11 to C12, D5 to D4, D6 to D5, D7 to D6
Connections:
- net +3.3V: now also C12.2, C18.2, L1.1; no longer C15.1
- net GND: now also C15.1, C16.1, C17.1, C19.1, C20.1, C21.1, D5.1 (K), C22.1, C23.1, C24.1; no longer C15.2, C16.2, C17.2, C19.2, C20.2, C21.2, J4.19 (VPP)
- net PREVGH: now also C19.2
- net PREVGL: now also C23.2
- net at J4.5 (VGH): now also C22.2; no longer C19.1
- net at J4.20 (VSH): now also C17.2; no longer C17.1
- net at J4.22 (VSL): now also C21.2; no longer C20.1
- net at J4.24 (VCOM): now also C24.2; no longer C21.1
- net at J4.4 (VGL): now also C20.2; no longer C18.2
- net D/C# renamed D/C
- net RES# renamed RES
- removed net VDD: C12.2, C16.1, J4.18 (VDD), L1.1
- new net: C15.2, J4.18 (VDD)
- new net: C16.2, J4.19 (VPP)
Other:
- moved on the sheet: C12, C13, C14, D4, D5, D6, R10, R11
